Commit message: gestione raccolta pomodori

File: husky_customization/husky_custom_description/urdf/custom_description.urdf.xacro (robot description, xacro)
@@ -26,17 +26,17 @@
   <xacro:arg name="kinect_enabled" default="false" />
   <xacro:include filename="$(find husky_description)/urdf/husky.urdf.xacro" />
-  <xacro:husky_robot />
+  <!-- <xacro:husky_robot /> -->
   <!-- Insert customization below, sample provided: -->
   <link name="bowler_link">
     <visual>
       <geometry>
-        <mesh filename="package://husky_custom_description/meshes/red_bowler.dae" />
+        <mesh filename="package://husky_custom_description/meshes/cassetta.dae" />
       </geometry>
     </visual>
     <collision>
-      <origin xyz="0 0 0.07" rpy="0 0 0" />
-      <geometry>
-        <box size="0.32 0.25 0.14" rpy="0 0 0"/>
-      </geometry>
+      <origin xyz="0 0 0" rpy="0 0 0" />
+       <geometry>
+           <mesh filename="package://husky_custom_description/meshes/cassetta.dae" />
+        </geometry>
     </collision>
   </link>
@@ -44,5 +44,5 @@
     <parent link="top_plate_link" />
     <child link="bowler_link" />
-    <origin xyz="0.1 -0.1 0" rpy="0 0 0.5" />
+    <origin xyz="-0.2 0 -0.2" rpy="0 0 0" />
   </joint>
 </robot>
